File: Electronics/BARBOT.sch (EAGLE design)
At the start: 59 parts, among them IC1 MEGA8-P, Q1 IRLR024, Q10 A03400, Q11 A03400, Q12 A03400, Q2 16MHZ

Commit message: CAD
Parts:
- removed Q10, Q11, Q12: A03400, SparkFun-DiscreteSemi:MOSFET-NCH-AO3404A
- removed R26, R29: 10R, rcl:R-US_R1206
- added D3: MBRA210LT3, microbuilder:DIODESMA
- added JP7: (no value), pinhead:PINHD-1X4
- added LED10, LED11, LED12, LED13, LED14, LED15, LED16, LED17, LED18, LED19, LED20, LED9: WS2812B5050, adafruit:WS2812B5050
- added Q3: IRLR024, Cohesion_parts:N-POWER-MOSFETDPAK-MOSFET
- D1: value 1N4148WS-SOD323 -> M4
- JP1, JP2, JP3: device pinhead:PINHD-1X4 -> pinhead:PINHD-1X3
Connections:
- net D10_MSFT3 renamed D10_MSFT_GOSWITCH
- net N$17 renamed LINK2
- net N$18 renamed LINK3
- net N$19 renamed LINK4
- net N$20 renamed LINK5
- net N$21 renamed LINK6
- net N$22 renamed LINK7
- net N$23 renamed LINK8
- net N$27 renamed LINK1
- removed net A2_SW2: C12.1, IC1.PC2(ADC2), JP2.2, R6.1
- removed net A3_SW3: C13.1, IC1.PC3(ADC3), JP1.2, R7.1
- removed net D10OUT_SW2: JP2.3, Q11.D
- removed net D13OUT_SW3: JP1.3, Q12.D
- removed net D13_MSFT4: IC1.PB5(SCK), R29.2
- removed net D9OUT_SW1: JP3.3, Q10.D
- removed net N$81: Q10.G, R26.1
- removed net N$83: Q12.G, R29.1
- new net 5V1: JP2.3, JP3.3, LED10.VDD, LED11.VDD, LED12.VDD, LED13.VDD, LED14.VDD, LED15.VDD, LED16.VDD, LED17.VDD, LED18.VDD, LED19.VDD, LED20.VDD, LED9.VDD
- new net A2_SW_SINGLE: C12.1, IC1.PC2(ADC2), JP1.1, R6.1
- new net A3_SW_DOUBLE: C13.1, IC1.PC3(ADC3), JP1.3, R7.1
- new net D10OUT_GOSWITCH: JP7.1, Q3.D
- new net D13: IC1.PB5(SCK)
- new net GND1: JP2.1, JP3.1, LED10.GND, LED11.GND, LED12.GND, LED13.GND, LED14.GND, LED15.GND, LED16.GND, LED17.GND, LED18.GND, LED19.GND, LED20.GND, LED9.GND
- new net LINK10: LED10.DI, LED9.DO
- new net LINK11: LED10.DO, LED11.DI
- new net LINK12: LED11.DO, LED12.DI
- new net LINK13: LED12.DO, LED13.DI
- new net LINK14: LED13.DO, LED14.DI
- new net LINK15: LED14.DO, LED15.DI
- new net LINK16: LED15.DO, LED16.DI
- new net LINK9: JP2.2, LED9.DI
- new net N$17: LED18.DO, LED19.DI
- new net N$18: LED19.DO, LED20.DI
- new net N$4: D3.A, J4.2
- new net N$6: JP3.2, LED20.DO
- new net N$7: LED16.DO, LED17.DI
- new net N$8: LED17.DO, LED18.DI
- net 24V: now also D3.C, JP7.4; no longer J4.2, JP1.4, JP2.4, JP3.4
- net A1_SW1: now also JP7.3; no longer JP3.2
- net D9_MSFT2: no longer R26.2
- net GND: now also JP1.2, JP7.2, Q3.S; no longer JP1.1, JP2.1, JP3.1, Q10.S, Q11.S, Q12.S
- net N$82: now also Q3.G; no longer Q11.G
Other:
- moved on the sheet: JP4, JP5
